File: IC-PDM-V2.1/IC-PDM-V2.1.kicad_pcb (KiCad board)
At the start: 2 copper layers, 118 x 78 mm, 47 parts, among them J1 RST, J10 Conn_01x04, J11 Conn_01x04, J12 Conn_01x04, J13 Conn_01x04, J14 Conn_01x04, J15 Conn_01x04, J16 Conn_01x02, J18 S03B-XASK-1, J2 BSEL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

Commit message: Ready to order
Parts:
- added G***: LOGO, LOGO, B.Cu at (199.8, 70.9)
- added REF**: jamesp-F.Cu, CustomFootprints:jamesp-F.Cu, F.Cu at (147.3, 99.3)
Other:
- board text added: "IC PDM V2.1 Designed by James Platt Routed 07/05/26"
