File: IC-PDM-V2.1/IC-PDM-V2.1.kicad_sch (KiCad schematic)
At the start: 46 parts, among them J1 RST, J10 Conn_01x04, J11 Conn_01x04, J12 Conn_01x04, J13 Conn_01x04, J14 Conn_01x04, J15 Conn_01x04, J16 Conn_01x02, J18 S03B-XASK-1, J2 BSEL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

Commit message: Ready to order
Connections:
- net +5V_Supply is gone; now on net +5V: U3.3 (FB)
Changed lines of the file:
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@@
 			)
 		)
-		(property "Value" "+5V_Supply"
+		(property "Value" "+5V"
 			(at 54.61 264.16 0)
 			(show_name no)
